File: Hardware/USB-C_Connector.kicad_sch (KiCad schematic)
At the start: 6 parts, among them J6 USB_C_Receptacle_USB2.0_16P

Commit message: Added TestPoints
Parts:
- C28: footprint Capacitor_SMD:C_0805_2012Metric -> Capacitor_SMD:C_0603_1608Metric_Pad1.08x0.95mm_HandSolder
Changed lines of the file:
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@@
 			)
 		)
-		(property "Footprint" "Capacitor_SMD:C_0805_2012Metric"
+		(property "Footprint" "Capacitor_SMD:C_0603_1608Metric_Pad1.08x0.95mm_HandSolder"
 			(at 66.3448 33.02 0)
 			(hide yes)

Commit message: Final Review Ready
Parts:
- added C41: 4.7nF, symbol Device:C
- added R11: 1M, symbol Device:R
Connections:
- net GND: now also C41.2, R11.2; no longer J6.S1 (SHIELD), J6.S2 (Shield), J6.S3 (Shield), J6.S4 (Shield)
- new net: C41.1, J6.S1 (SHIELD), J6.S2 (Shield), J6.S3 (Shield), J6.S4 (Shield), R11.1
