File: Hardware/linpot.kicad_sch (KiCad schematic)
At the start: 6 parts, among them U6 Opamp_Dual

Commit message: fixed some subsheets
Parts:
- added C25: 1u, symbol Device:C
- R25: value 0 -> 4.7k; footprint (none) -> LHRS_Connectors:Molex_Nano-Fit_105309-xx05_1x05_P2.50mm_Vertical; P/N CRCW06030000Z0EE -> (none)
- renumbered C42 to C46, C43 to C47, D12 to D13, F2 to F3, U6 to U7
Connections:
- net LinPot_Signal: now also R25.2; no longer D13.1 (A1), U7.2 (-)
- net GND renamed GNDA
- net GNDA: now also C25.2; no longer R25.2
- net SHIELD renamed LinPot_Output
- net LinPot_Output: now also D13.1 (A1), U7.2 (-), C25.1
Other:
- moved on the sheet: F3

Commit message: made review changes
Other:
- moved on the sheet: C25, C46, C47, D13, F3, R25, U7A, U7B, U7C

Commit message: Added TestPoints
Parts:
- C25: value 1u -> 1uF; footprint (none) -> Capacitor_SMD:C_0603_1608Metric_Pad1.08x0.95mm_HandSolder
- C46: value 100n -> 100nF; footprint (none) -> Capacitor_SMD:C_0603_1608Metric_Pad1.08x0.95mm_HandSolder
- C47: value 10u -> 10uF; footprint (none) -> Capacitor_SMD:C_0603_1608Metric_Pad1.08x0.95mm_HandSolder
Changed lines of the file:
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@@
 	)
 	(image
-		(at 90.17 158.75)
+		(at 88.9 105.41)
 		(data "iVBORw0KGgoAAAANSUhEUgAABfQAAAJKCAIAAADlRVPHAAAAA3NCSVQICAjb4U/gAAAgAElEQVR4"
 			"nOzdd1xW5f/H8euc+2ZPBXErThD31gTTRNFc5dYsU7Nlan3r59ZMzXCPhlpmVqaVmiMVBXEP3BvR"
@@
 	)
 	(hierarchical_label "GNDA"
-		(shape input)
+		(shape bidirectional)
 		(at 190.5 55.88 0)
 		(effects
@@
 	)
 	(hierarchical_label "GNDA"
-		(shape input)
+		(shape bidirectional)
 		(at 228.6 68.58 270)
 		(effects
@@
 	)
 	(hierarchical_label "GNDA"
-		(shape input)
+		(shape bidirectional)
 		(at 160.02 60.96 0)
 		(effects
@@
 			)
 		)
-		(property "Value" "100n"
+		(property "Value" "100nF"
 			(at 237.744 58.42 0)
 			(show_name no)
@@
 			)
 		)
-		(property "Footprint" ""
+		(property "Footprint" "Capacitor_SMD:C_0603_1608Metric_Pad1.08x0.95mm_HandSolder"
 			(at 233.9848 53.34 0)
 			(hide yes)
@@
 			)
 		)
-		(property "Value" "10u"
+		(property "Value" "10uF"
 			(at 247.904 58.42 0)
 			(show_name no)
@@
 			)
 		)
-		(property "Footprint" ""
+		(property "Footprint" "Capacitor_SMD:C_0603_1608Metric_Pad1.08x0.95mm_HandSolder"
 			(at 244.1448 53.34 0)
 			(hide yes)
@@
 			)
 		)
-		(property "Value" "1u"
+		(property "Value" "1uF"
 			(at 189.484 54.102 90)
 			(show_name no)
@@
 			)
 		)
-		(property "Footprint" ""
+		(property "Footprint" "Capacitor_SMD:C_0603_1608Metric_Pad1.08x0.95mm_HandSolder"
 			(at 189.23 54.9148 0)
 			(hide yes)

Commit message: Final Review Ready
Parts:
- D13: value D_TVS -> TVS; footprint Diode_SMD:Nexperia_DSN1608-2_1.6x0.8mm -> Diode_SMD:D_SOD-323_HandSoldering
Changed lines of the file:
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@@
 			)
 		)
-		(property "Value" "D_TVS"
+		(property "Value" "TVS"
 			(at 160.02 58.4199 90)
 			(show_name no)
@@
 			)
 		)
-		(property "Footprint" "Diode_SMD:Nexperia_DSN1608-2_1.6x0.8mm"
+		(property "Footprint" "Diode_SMD:D_SOD-323_HandSoldering"
 			(at 157.48 57.15 0)
 			(hide yes)
@@
 			)
 		)
-		(property "Datasheet" ""
+		(property "Datasheet" "kicad-embed://TVS.pdf"
 			(at 157.48 57.15 0)
 			(hide yes)
@@
 			)
 		)
-		(property "Datasheet" ""
+		(property "Datasheet" "https://www.ti.com/lit/ds/symlink/tlv9001-q1.pdf?ts=1791336000098&ref_url=https%253A%252F%252Fwww.mouser.com%252F"
 			(at 147.32 48.26 0)
 			(hide yes)
@@
 			)
 		)
-		(property "Datasheet" ""
+		(property "Datasheet" "https://www.ti.com/lit/ds/symlink/tlv9001-q1.pdf?ts=1791336000098&ref_url=https%253A%252F%252Fwww.mouser.com%252F"
 			(at 243.84 86.36 0)
 			(hide yes)
@@
 			)
 		)
-		(property "Datasheet" ""
+		(property "Datasheet" "https://www.ti.com/lit/ds/symlink/tlv9001-q1.pdf?ts=1791336000098&ref_url=https%253A%252F%252Fwww.mouser.com%252F"
 			(at 231.14 57.15 0)
 			(hide yes)

Commit message: Final Changes before Final Review
Other:
- moved on the sheet: C47
Changed lines of the file:
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@@
 	(wire
 		(pts
-			(xy 245.11 49.53) (xy 245.11 53.34)
+			(xy 246.38 49.53) (xy 246.38 53.34)
 		)
 		(stroke
@@
 	(wire
 		(pts
-			(xy 245.11 60.96) (xy 245.11 66.04)
+			(xy 246.38 60.96) (xy 246.38 66.04)
 		)
 		(stroke
@@
 	(wire
 		(pts
-			(xy 234.95 49.53) (xy 245.11 49.53)
+			(xy 234.95 49.53) (xy 246.38 49.53)
 		)
 		(stroke
@@
 	(wire
 		(pts
-			(xy 245.11 66.04) (xy 234.95 66.04)
+			(xy 246.38 66.04) (xy 234.95 66.04)
 		)
 		(stroke
@@
 	(symbol
 		(lib_id "Device:C")
-		(at 245.11 57.15 180)
+		(at 246.38 57.15 180)
 		(unit 1)
 		(body_style 1)
@@
 		(dnp no)
 		(property "Reference" "C47"
-			(at 247.904 55.88 0)
+			(at 249.174 55.88 0)
 			(show_name no)
 			(do_not_autoplace no)
@@
 		)
 		(property "Value" "10uF"
-			(at 247.904 58.42 0)
+			(at 249.174 58.42 0)
 			(show_name no)
 			(do_not_autoplace no)
@@
 		)
 		(property "Footprint" "Capacitor_SMD:C_0603_1608Metric_Pad1.08x0.95mm_HandSolder"
-			(at 244.1448 53.34 0)
+			(at 245.4148 53.34 0)
 			(hide yes)
 			(show_name no)
@@
 		)
 		(property "Datasheet" ""
-			(at 245.11 57.15 0)
+			(at 246.38 57.15 0)
 			(hide yes)
 			(show_name no)
@@
 		)
 		(property "Description" "Unpolarized capacitor"
-			(at 245.11 57.15 0)
+			(at 246.38 57.15 0)
 			(hide yes)
 			(show_name no)
@@
 		)
 		(property "P/N" "GRM21BR61H106KE43L"
-			(at 245.11 57.15 0)
-			(hide yes)
-			(show_name no)
+			(at 246.38 57.15 0)
+			(hide yes)
+			(show_name no)

Commit message: Final Review Ready
Changed lines of the file:
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@@
 	(wire
 		(pts
-			(xy 170.18 48.26) (xy 171.45 48.26)
+			(xy 168.91 48.26) (xy 171.45 48.26)
 		)
 		(stroke
@@
 	(hierarchical_label "LinPot_Output"
 		(shape output)
-		(at 170.18 48.26 180)
+		(at 168.91 48.26 180)
 		(effects
 			(font
@@
 		)
 		(property "Value" "1uF"
-			(at 189.484 54.102 90)
-			(show_name no)
-			(do_not_autoplace no)
+			(at 183.642 57.15 90)
+			(show_name no)
+			(do_not_autoplace no)

Commit message: Updated KiCAD Sharepoint
Connections:
- net AMP_LinPot: now also U7.2 (-); no longer U7.3 (+)
- net LinPot_Output: now also U7.3 (+); no longer U7.2 (-)
Other:
- note added: "Cutoff: 34Hz"
- moved on the sheet: C25, C46, D13, F3, R25, U7A, U7B, U7C
