File: Hardware/CAN_Transceiver.kicad_sch (KiCad schematic)
At the start: 9 parts, among them IC1 TCAN3413DR

Commit message: Refactored Schematic to use SubSheets
Parts:
- renumbered C24 to C40, C25 to C41, C26 to C44, C27 to C45, D6 to D11, IC1 to IC3, JP1 to JP2, R11 to R24, R12 to R26
Changed lines of the file:
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@@
 		(in_pos_files yes)
 		(dnp no)
-		(property "Reference" "C25"
+		(property "Reference" "C41"
 			(at 76.2 73.66 0)
 			(show_name no)
@@
 		)
 		(instances
-			(project ""
-				(path "/69b823fd-c065-40ff-9bb9-c5835555f3eb/9d9eae1e-c713-4323-9845-a569cff8d5d3"
-					(reference "C6")
-					(unit 1)
-				)
-			)
-			(project "CAN_Transceiver"
-				(path "/a09f9696-80ee-4697-8aaa-225f287b667b"
-					(reference "C2")
-					(unit 1)
-				)
-			)
 			(project "SuspensionBoard"
-				(path "/f9dc491a-b8c6-4623-9728-13837ac4bba3/963419ad-288c-4ad7-963b-cb6fd15ddb22"
-					(reference "C25")
+				(path "/f9dc491a-b8c6-4623-9728-13837ac4bba3/d2e121da-4655-471c-894c-244db72f6066/5cd0492a-8586-4c19-a808-4d3883e80abc"
+					(reference "C41")
 					(unit 1)
 				)
@@
 		(in_pos_files yes)
 		(dnp no)
-		(property "Reference" "C27"
+		(property "Reference" "C45"
 			(at 194.564 88.646 0)
 			(show_name no)
@@
 		)
 		(instances
-			(project ""
-				(path "/69b823fd-c065-40ff-9bb9-c5835555f3eb/9d9eae1e-c713-4323-9845-a569cff8d5d3"
-					(reference "C8")
-					(unit 1)
-				)
-			)
-			(project "CAN_Transceiver"
-				(path "/a09f9696-80ee-4697-8aaa-225f287b667b"
-					(reference "C4")
-					(unit 1)
-				)
-			)
 			(project "SuspensionBoard"
-				(path "/f9dc491a-b8c6-4623-9728-13837ac4bba3/963419ad-288c-4ad7-963b-cb6fd15ddb22"
-					(reference "C27")
+				(path "/f9dc491a-b8c6-4623-9728-13837ac4bba3/d2e121da-4655-471c-894c-244db72f6066/5cd0492a-8586-4c19-a808-4d3883e80abc"
+					(reference "C45")
 					(unit 1)
 				)
@@
 		(dnp no)
 		(fields_autoplaced yes)
-		(property "Reference" "JP1"
+		(property "Reference" "JP2"
 			(at 215.9 78.74 0)
 			(show_name no)
@@
 		)
 		(instances
-			(project ""
-				(path "/69b823fd-c065-40ff-9bb9-c5835555f3eb/9d9eae1e-c713-4323-9845-a569cff8d5d3"
+			(project "SuspensionBoard"
+				(path "/f9dc491a-b8c6-4623-9728-13837ac4bba3/d2e121da-4655-471c-894c-244db72f6066/5cd0492a-8586-4c19-a808-4d3883e80abc"
 					(reference "JP2")
-					(unit 1)
-				)
-			)
-			(project ""
-				(path "/81d906df-a099-480a-8398-28a8e913d125"
-					(reference "JP1")
-					(unit 1)
-				)
-			)
-			(project "CAN_Transceiver"
-				(path "/a09f9696-80ee-4697-8aaa-225f287b667b"
-					(reference "JP1")
-					(unit 1)
-				)
-			)
-			(project "SuspensionBoard"
-				(path "/f9dc491a-b8c6-4623-9728-13837ac4bba3/963419ad-288c-4ad7-963b-cb6fd15ddb22"
-					(reference "JP1")
 					(unit 1)
 				)
@@
 		(in_pos_files yes)
 		(dnp no)
-		(property "Reference" "C26"
+		(property "Reference" "C44"
 			(at 88.138 73.66 0)
 			(show_name no)
@@
 		)
 		(instances
-			(project ""
-				(path "/69b823fd-c065-40ff-9bb9-c5835555f3eb/9d9eae1e-c713-4323-9845-a569cff8d5d3"
-					(reference "C7")
-					(unit 1)
-				)
-			)
-			(project "CAN_Transceiver"
-				(path "/a09f9696-80ee-4697-8aaa-225f287b667b"
-					(reference "C3")
-					(unit 1)
-				)
-			)
 			(project "SuspensionBoard"
-				(path "/f9dc491a-b8c6-4623-9728-13837ac4bba3/963419ad-288c-4ad7-963b-cb6fd15ddb22"
-					(reference "C26")
+				(path "/f9dc491a-b8c6-4623-9728-13837ac4bba3/d2e121da-4655-471c-894c-244db72f6066/5cd0492a-8586-4c19-a808-4d3883e80abc"
+					(reference "C44")
 					(unit 1)
 				)
@@
 		(in_pos_files yes)
 		(dnp no)
-		(property "Reference" "C24"
+		(property "Reference" "C40"
 			(at 65.278 73.66 0)
 			(show_name no)
@@
 		)
 		(instances
-			(project ""
-				(path "/69b823fd-c065-40ff-9bb9-c5835555f3eb/9d9eae1e-c713-4323-9845-a569cff8d5d3"
-					(reference "C5")
-					(unit 1)
-				)
-			)
-			(project ""
-				(path "/81d906df-a099-480a-8398-28a8e913d125"
-					(reference "C1")
-					(unit 1)
-				)
-			)
-			(project "CAN_Transceiver"
-				(path "/a09f9696-80ee-4697-8aaa-225f287b667b"
-					(reference "C1")
-					(unit 1)
-				)
-			)
 			(project "SuspensionBoard"
-				(path "/f9dc491a-b8c6-4623-9728-13837ac4bba3/963419ad-288c-4ad7-963b-cb6fd15ddb22"
-					(reference "C24")
+				(path "/f9dc491a-b8c6-4623-9728-13837ac4bba3/d2e121da-4655-471c-894c-244db72f6066/5cd0492a-8586-4c19-a808-4d3883e80abc"
+					(reference "C40")
 					(unit 1)
 				)
@@
 		(in_pos_files yes)
 		(dnp no)
-		(property "Reference" "R12"
+		(property "Reference" "R26"
 			(at 201.93 80.01 90)
 			(show_name no)
@@
 		)
 		(instances
-			(project "kk36984"
-				(path "/69b823fd-c065-40ff-9bb9-c5835555f3eb/9d9eae1e-c713-4323-9845-a569cff8d5d3"
-					(reference "R23")
-					(unit 1)
-				)
-			)
-			(project "CAN_Transceiver"
-				(path "/a09f9696-80ee-4697-8aaa-225f287b667b"
-					(reference "R2")
-					(unit 1)
-				)
-			)
 			(project "SuspensionBoard"
-				(path "/f9dc491a-b8c6-4623-9728-13837ac4bba3/963419ad-288c-4ad7-963b-cb6fd15ddb22"
-					(reference "R12")
+				(path "/f9dc491a-b8c6-4623-9728-13837ac4bba3/d2e121da-4655-471c-894c-244db72f6066/5cd0492a-8586-4c19-a808-4d3883e80abc"
+					(reference "R26")
 					(unit 1)
 				)
@@
 		(dnp no)
 		(fields_autoplaced yes)
-		(property "Reference" "D6"
+		(property "Reference" "D11"
 			(at 196.85 46.99 0)
 			(show_name no)
@@
 		)
 		(instances
-			(project ""
-				(path "/69b823fd-c065-40ff-9bb9-c5835555f3eb/9d9eae1e-c713-4323-9845-a569cff8d5d3"
-					(reference "D8")
-					(unit 1)
-				)
-			)
-			(project "CAN_Transceiver"
-				(path "/a09f9696-80ee-4697-8aaa-225f287b667b"
-					(reference "D1")
-					(unit 1)
-				)
-			)
 			(project "SuspensionBoard"
-				(path "/f9dc491a-b8c6-4623-9728-13837ac4bba3/963419ad-288c-4ad7-963b-cb6fd15ddb22"
-					(reference "D6")
+				(path "/f9dc491a-b8c6-4623-9728-13837ac4bba3/d2e121da-4655-471c-894c-244db72f6066/5cd0492a-8586-4c19-a808-4d3883e80abc"
+					(reference "D11")
 					(unit 1)
 				)
@@
 		(dnp no)
 		(fields_autoplaced yes)
-		(property "Reference" "IC1"
+		(property "Reference" "IC3"
 			(at 128.27 63.5 0)
 			(show_name no)
@@
 		)
 		(instances
-			(project ""
-				(path "/69b823fd-c065-40ff-9bb9-c5835555f3eb/9d9eae1e-c713-4323-9845-a569cff8d5d3"
-					(reference "IC1")
-					(unit 1)
-				)
-			)
-			(project "CAN_Transceiver"
-				(path "/a09f9696-80ee-4697-8aaa-225f287b667b"
-					(reference "IC1")
-					(unit 1)
-				)
-			)
 			(project "SuspensionBoard"
-				(path "/f9dc491a-b8c6-4623-9728-13837ac4bba3/963419ad-288c-4ad7-963b-cb6fd15ddb22"
-					(reference "IC1")
+				(path "/f9dc491a-b8c6-4623-9728-13837ac4bba3/d2e121da-4655-471c-894c-244db72f6066/5cd0492a-8586-4c19-a808-4d3883e80abc"
+					(reference "IC3")
 					(unit 1)
 				)
@@
 		(in_pos_files yes)
 		(dnp no)
-		(property "Reference" "R11"
+		(property "Reference" "R24"
 			(at 176.53 80.01 90)
 			(show_name no)
@@
 		)
 		(instances
-			(project ""
-				(path "/69b823fd-c065-40ff-9bb9-c5835555f3eb/9d9eae1e-c713-4323-9845-a569cff8d5d3"
-					(reference "R22")
+			(project "SuspensionBoard"
+				(path "/f9dc491a-b8c6-4623-9728-13837ac4bba3/d2e121da-4655-471c-894c-244db72f6066/5cd0492a-8586-4c19-a808-4d3883e80abc"
+					(reference "R24")
 					(unit 1)
 				)
-			)
-			(project ""
-				(path "/81d906df-a099-480a-8398-28a8e913d125"
-					(reference "R1")
-					(unit 1)
-				)
-			)
-			(project "CAN_Transceiver"
-				(path "/a09f9696-80ee-4697-8aaa-225f287b667b"
-					(reference "R1")
-					(unit 1)
-				)
-			)
-			(project "SuspensionBoard"
-				(path "/f9dc491a-b8c6-4623-9728-13837ac4bba3/963419ad-288c-4ad7-963b-cb6fd15ddb22"
-					(reference "R11")
-					(unit 1)
-				)

Commit message: made review changes
Parts:
- renumbered C40 to C24, C41 to C26, C44 to C27, C45 to C40, D11 to D6, IC3 to IC1, JP2 to JP1
Changed lines of the file:
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@@
 	(text "CAN Transceiver\n"
 		(exclude_from_sim no)
-		(at 69.596 49.784 0)
+		(at 69.85 49.53 0)
 		(effects
 			(font
@@
 	(text "Try to keep CDSOT23 near bus conn"
 		(exclude_from_sim no)
-		(at 197.866 64.008 0)
+		(at 198.12 63.5 0)
 		(effects
 			(font
@@
 	(text "CAN Protection"
 		(exclude_from_sim no)
-		(at 177.546 43.942 0)
+		(at 177.8 44.45 0)
 		(effects
 			(font
@@
 	(text "CAN Bus Termination\n"
 		(exclude_from_sim no)
-		(at 181.864 76.454 0)
+		(at 181.61 76.2 0)
 		(effects
 			(font
@@
 		(in_pos_files yes)
 		(dnp no)
-		(property "Reference" "C41"
+		(property "Reference" "C26"
 			(at 76.2 73.66 0)
 			(show_name no)
@@
 		(instances
 			(project "SuspensionBoard"
-				(path "/f9dc491a-b8c6-4623-9728-13837ac4bba3/d2e121da-4655-471c-894c-244db72f6066/5cd0492a-8586-4c19-a808-4d3883e80abc"
-					(reference "C41")
+				(path "/f9dc491a-b8c6-4623-9728-13837ac4bba3/5db358c0-18b3-459f-8665-95f1e3ffe97b"
+					(reference "C26")
 					(unit 1)
 				)
@@
 		(in_pos_files yes)
 		(dnp no)
-		(property "Reference" "C45"
+		(property "Reference" "C40"
 			(at 194.564 88.646 0)
 			(show_name no)
@@
 		(instances
 			(project "SuspensionBoard"
-				(path "/f9dc491a-b8c6-4623-9728-13837ac4bba3/d2e121da-4655-471c-894c-244db72f6066/5cd0492a-8586-4c19-a808-4d3883e80abc"
-					(reference "C45")
+				(path "/f9dc491a-b8c6-4623-9728-13837ac4bba3/5db358c0-18b3-459f-8665-95f1e3ffe97b"
+					(reference "C40")
 					(unit 1)
 				)
@@
 		(dnp no)
 		(fields_autoplaced yes)
-		(property "Reference" "JP2"
+		(property "Reference" "JP1"
 			(at 215.9 78.74 0)
 			(show_name no)
@@
 		(instances
 			(project "SuspensionBoard"
-				(path "/f9dc491a-b8c6-4623-9728-13837ac4bba3/d2e121da-4655-471c-894c-244db72f6066/5cd0492a-8586-4c19-a808-4d3883e80abc"
-					(reference "JP2")
+				(path "/f9dc491a-b8c6-4623-9728-13837ac4bba3/5db358c0-18b3-459f-8665-95f1e3ffe97b"
+					(reference "JP1")
 					(unit 1)
 				)
@@
 		(in_pos_files yes)
 		(dnp no)
-		(property "Reference" "C44"
+		(property "Reference" "C27"
 			(at 88.138 73.66 0)
 			(show_name no)
@@
 		(instances
 			(project "SuspensionBoard"
-				(path "/f9dc491a-b8c6-4623-9728-13837ac4bba3/d2e121da-4655-471c-894c-244db72f6066/5cd0492a-8586-4c19-a808-4d3883e80abc"
-					(reference "C44")
+				(path "/f9dc491a-b8c6-4623-9728-13837ac4bba3/5db358c0-18b3-459f-8665-95f1e3ffe97b"
+					(reference "C27")
 					(unit 1)
 				)
@@
 		(in_pos_files yes)
 		(dnp no)
-		(property "Reference" "C40"
+		(property "Reference" "C24"
 			(at 65.278 73.66 0)
 			(show_name no)
@@
 		(instances
 			(project "SuspensionBoard"
-				(path "/f9dc491a-b8c6-4623-9728-13837ac4bba3/d2e121da-4655-471c-894c-244db72f6066/5cd0492a-8586-4c19-a808-4d3883e80abc"
-					(reference "C40")
+				(path "/f9dc491a-b8c6-4623-9728-13837ac4bba3/5db358c0-18b3-459f-8665-95f1e3ffe97b"
+					(reference "C24")
 					(unit 1)
 				)
@@
 		(dnp no)
 		(property "Reference" "R26"
-			(at 201.93 80.01 90)
+			(at 201.93 83.058 90)
 			(show_name no)
 			(do_not_autoplace no)
@@
 		)
 		(property "Value" "60"
-			(at 201.93 82.55 90)
+			(at 201.93 85.09 90)
 			(show_name no)
 			(do_not_autoplace no)
@@
 		(instances
 			(project "SuspensionBoard"
-				(path "/f9dc491a-b8c6-4623-9728-13837ac4bba3/d2e121da-4655-471c-894c-244db72f6066/5cd0492a-8586-4c19-a808-4d3883e80abc"
+				(path "/f9dc491a-b8c6-4623-9728-13837ac4bba3/5db358c0-18b3-459f-8665-95f1e3ffe97b"
 					(reference "R26")
 					(unit 1)
@@
 		(dnp no)
 		(fields_autoplaced yes)
-		(property "Reference" "D11"
+		(property "Reference" "D6"
 			(at 196.85 46.99 0)
 			(show_name no)
@@
 		(instances
 			(project "SuspensionBoard"
-				(path "/f9dc491a-b8c6-4623-9728-13837ac4bba3/d2e121da-4655-471c-894c-244db72f6066/5cd0492a-8586-4c19-a808-4d3883e80abc"
-					(reference "D11")
+				(path "/f9dc491a-b8c6-4623-9728-13837ac4bba3/5db358c0-18b3-459f-8665-95f1e3ffe97b"
+					(reference "D6")
 					(unit 1)
 				)
@@
 		(dnp no)
 		(fields_autoplaced yes)
-		(property "Reference" "IC3"
+		(property "Reference" "IC1"
 			(at 128.27 63.5 0)
 			(show_name no)
@@
 		(instances
 			(project "SuspensionBoard"
-				(path "/f9dc491a-b8c6-4623-9728-13837ac4bba3/d2e121da-4655-471c-894c-244db72f6066/5cd0492a-8586-4c19-a808-4d3883e80abc"
-					(reference "IC3")
+				(path "/f9dc491a-b8c6-4623-9728-13837ac4bba3/5db358c0-18b3-459f-8665-95f1e3ffe97b"
+					(reference "IC1")
 					(unit 1)
 				)
@@
 		(dnp no)
 		(property "Reference" "R24"
-			(at 176.53 80.01 90)
+			(at 176.53 83.058 90)
 			(show_name no)
 			(do_not_autoplace no)
@@
 		)
 		(property "Value" "60"
-			(at 176.53 82.55 90)
+			(at 176.53 85.09 90)
 			(show_name no)
 			(do_not_autoplace no)
@@
 		(instances
 			(project "SuspensionBoard"
-				(path "/f9dc491a-b8c6-4623-9728-13837ac4bba3/d2e121da-4655-471c-894c-244db72f6066/5cd0492a-8586-4c19-a808-4d3883e80abc"
+				(path "/f9dc491a-b8c6-4623-9728-13837ac4bba3/5db358c0-18b3-459f-8665-95f1e3ffe97b"
 					(reference "R24")
 					(unit 1)

Commit message: Added TestPoints
Parts:
- C24: value 10u -> 10uF; footprint Capacitor_SMD:C_0805_2012Metric_Pad1.18x1.45mm_HandSolder -> Capacitor_SMD:C_0603_1608Metric_Pad1.08x0.95mm_HandSolder
- C26, C27, C40: value 0.1u -> 0.1uF
Changed lines of the file:
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@@
 			)
 		)
-		(property "Value" "0.1u"
+		(property "Value" "0.1uF"
 			(at 75.946 75.946 0)
 			(show_name no)
@@
 			)
 		)
-		(property "Value" "0.1u"
+		(property "Value" "0.1uF"
 			(at 194.564 91.186 0)
 			(show_name no)
@@
 			)
 		)
-		(property "Value" "0.1u"
+		(property "Value" "0.1uF"
 			(at 88.138 76.2 0)
 			(show_name no)
@@
 			)
 		)
-		(property "Value" "10u"
+		(property "Value" "10uF"
 			(at 65.278 76.2 0)
 			(show_name no)
@@
 			)
 		)
-		(property "Footprint" "Capacitor_SMD:C_0805_2012Metric_Pad1.18x1.45mm_HandSolder"
+		(property "Footprint" "Capacitor_SMD:C_0603_1608Metric_Pad1.08x0.95mm_HandSolder"
 			(at 63.1952 78.74 0)
 			(hide yes)

Commit message: Made some changes
Parts:
- C24: value 10uF -> 10u; footprint Capacitor_SMD:C_0603_1608Metric_Pad1.08x0.95mm_HandSolder -> Capacitor_SMD:C_0805_2012Metric_Pad1.18x1.45mm_HandSolder
- C26, C27, C40: value 0.1uF -> 0.1u
- D5: renamed from D6; Height 1.17 -> (none); Manufacturer_Name Bourns -> (none); Mouser Part Number 652-CDSOT23-T24CAN -> (none); Mouser Price/Stock https://www.mouser.co.uk/ProductDetail/Bourns/CDSOT23-T24CA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 -> (none)
- IC1: Height 1.75 -> (none); Manufacturer_Name Texas Instruments -> (none); Mouser Part Number 595-TCAN3413DR -> (none); Mouser Price/Stock - -> (none)
Connections:
- net 3.3v renamed 3V3
