File: Hardware/PowerProtection.kicad_sch (KiCad schematic)
At the start: 18 parts, among them IC2 LM74502DDFR, Q1 PSMN012-100YS, Q2 PSMN012-100YS

Commit message: Added TestPoints
Parts:
- C29, C34, C35: value 0.1u -> 0.1uF
- C30: value 1u -> 1uF
- C31: value 220n -> 220nF
- C32: value 10n -> 10uF
- C33: value 10u -> 10uF; footprint Capacitor_SMD:C_0805_2012Metric_Pad1.18x1.45mm_HandSolder -> Capacitor_SMD:C_0603_1608Metric_Pad1.08x0.95mm_HandSolder
Changed lines of the file:
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@@
 			)
 		)
-		(property "Value" "220n"
+		(property "Value" "220nF"
 			(at 57.785 82.5499 0)
 			(show_name no)
@@
 			)
 		)
-		(property "Value" "0.1u"
+		(property "Value" "0.1uF"
 			(at 38.1 52.0699 0)
 			(show_name no)
@@
 			)
 		)
-		(property "Value" "0.1u"
+		(property "Value" "0.1uF"
 			(at 113.03 91.44 0)
 			(show_name no)
@@
 			)
 		)
-		(property "Value" "10n"
+		(property "Value" "10uF"
 			(at 54.61 64.262 0)
 			(show_name no)
@@
 			)
 		)
-		(property "Value" "10u"
+		(property "Value" "10uF"
 			(at 112.395 52.0699 0)
 			(show_name no)
@@
 			)
 		)
-		(property "Footprint" "Capacitor_SMD:C_0805_2012Metric_Pad1.18x1.45mm_HandSolder"
+		(property "Footprint" "Capacitor_SMD:C_0603_1608Metric_Pad1.08x0.95mm_HandSolder"
 			(at 110.1852 54.61 0)
 			(hide yes)
@@
 			)
 		)
-		(property "Value" "1u"
+		(property "Value" "1uF"
 			(at 31.75 85.0899 0)
 			(show_name no)
@@
 			)
 		)
-		(property "Value" "0.1u"
+		(property "Value" "0.1uF"
 			(at 131.826 91.44 0)
 			(show_name no)

Commit message: Made some changes
Parts:
- C29, C34, C35: value 0.1uF -> 0.1u
- C30: value 1uF -> 1u
- C31: value 220nF -> 220n
- C32: value 10uF -> 10n
- C33: value 10uF -> 10u; footprint Capacitor_SMD:C_0603_1608Metric_Pad1.08x0.95mm_HandSolder -> Capacitor_SMD:C_0805_2012Metric_Pad1.18x1.45mm_HandSolder
- IC2: Manufacturer_Name Texas Instruments -> (none); Manufacturer_Part_Number LM74502DDFR -> (none); Mouser Part Number 595-LM74502DDFR -> (none); Mouser Price/Stock https://www.mouser.co.uk/ProductDetail/Texas-Instruments/LM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 -> (none)
- R15, R17, R18, R19, R20: symbol Device:R_US -> Device:R
- R16: symbol Device:R_US -> Device:R; Mouser Part Number 594-MCT06030C3309FP5 -> (none)
- renumbered D9 to D6, D10 to D9
Other:
- note added: "Supp Battery Range: 10V-14.7V"
