File: Hardware/Power_Mux.kicad_sch (KiCad schematic)
At the start: 6 parts, among them U5 TPS2117DRLR

Commit message: made review changes
Changed lines of the file:
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@@
 	(text "Max and min threshold voltage calculations for 3v3 and 5v\n[delete this if you want :^)]"
 		(exclude_from_sim no)
-		(at 54.864 106.934 0)
+		(at 54.61 106.68 0)
 		(effects
 			(font
@@
 	(text "R2"
 		(exclude_from_sim no)
-		(at 31.75 68.834 0)
+		(at 31.75 68.58 0)
 		(effects
 			(font
@@
 	(text "R1"
 		(exclude_from_sim no)
-		(at 31.75 61.214 0)
+		(at 31.75 60.96 0)
 		(effects
 			(font
@@
 	(text "5v "
 		(exclude_from_sim no)
-		(at 58.42 115.316 0)
+		(at 58.42 115.57 0)
 		(effects
 			(font
@@
 	(text "Configured to use automatic switching mode: VIN_1 is prioritized"
 		(exclude_from_sim no)
-		(at 47.498 29.464 0)
+		(at 46.99 29.21 0)
 		(effects
 			(font
@@
 	(text "Acceptable input range is 1.6 to 5.5 volts\nResistor divider needs to be tuned depending on input\n"
 		(exclude_from_sim no)
-		(at 48.006 36.068 0)
+		(at 48.26 35.56 0)
 		(effects
 			(font
@@
 	(text "Resistor divider to meet Vref \nUser needs to set resistors!\nExample values:\nFor 5v:  R1 = 16k R2 = 4.7k   (Max threshold = 4.76, min = 4.05)\nFor 3v3: R1 = 18k R2 = 10k   (Max threshold = 3.02, min = 2.58)"
 		(exclude_from_sim no)
-		(at 16.002 87.376 0)
+		(at 16.51 87.63 0)
 		(effects
 			(font
@@
 	(text "5V/3V3 Power Mux"
 		(exclude_from_sim no)
-		(at 51.816 20.574 0)
+		(at 52.07 20.32 0)
 		(effects
 			(font

Commit message: Made some changes
Parts:
- C36, C37, C38, C39: value 0.1uF -> 0.1u; Mfg MLASH168SB7104KTNA01 -> (none)
- U4: renamed from U5; MANUFACTURER Texas Instruments -> (none); MAXIMUM_PACKAGE_HEIGHT 0.6mm -> (none); PARTREV A -> (none); STANDARD IPC-7351B -> (none)
Changed lines of the file:
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@@
 	(text "Max and min threshold voltage calculations for 3v3 and 5v\n[delete this if you want :^)]"
 		(exclude_from_sim no)
-		(at 54.61 106.68 0)
+		(at 54.864 106.934 0)
 		(effects
 			(font
@@
 	(text "R2"
 		(exclude_from_sim no)
-		(at 31.75 68.58 0)
+		(at 31.75 68.834 0)
 		(effects
 			(font
@@
 	(text "R1"
 		(exclude_from_sim no)
-		(at 31.75 60.96 0)
+		(at 31.75 61.214 0)
 		(effects
 			(font
@@
 	(text "5v "
 		(exclude_from_sim no)
-		(at 58.42 115.57 0)
+		(at 58.42 115.316 0)
 		(effects
 			(font
@@
 	(text "Configured to use automatic switching mode: VIN_1 is prioritized"
 		(exclude_from_sim no)
-		(at 46.99 29.21 0)
+		(at 47.498 29.464 0)
 		(effects
 			(font
@@
 	(text "Acceptable input range is 1.6 to 5.5 volts\nResistor divider needs to be tuned depending on input\n"
 		(exclude_from_sim no)
-		(at 48.26 35.56 0)
+		(at 48.006 36.068 0)
 		(effects
 			(font
@@
 	(text "Resistor divider to meet Vref \nUser needs to set resistors!\nExample values:\nFor 5v:  R1 = 16k R2 = 4.7k   (Max threshold = 4.76, min = 4.05)\nFor 3v3: R1 = 18k R2 = 10k   (Max threshold = 3.02, min = 2.58)"
 		(exclude_from_sim no)
-		(at 16.51 87.63 0)
+		(at 16.002 87.376 0)
 		(effects
 			(font
@@
 	(text "5V/3V3 Power Mux"
 		(exclude_from_sim no)
-		(at 52.07 20.32 0)
+		(at 51.816 20.574 0)
 		(effects
 			(font
@@
 			)
 		)
-		(property "Value" "0.1uF"
+		(property "Value" "0.1u"
 			(at 91.8972 59.563 0)
 			(show_name no)
@@
 			)
 		)
-		(property "Mfg" "MLASH168SB7104KTNA01"
-			(at 88.9 58.42 0)
-			(hide yes)
-			(show_name no)
-			(do_not_autoplace no)
-			(effects
-				(font
-					(size 1.27 1.27)
-				)
-			)
-		)
 		(pin "1"
 		)
@@
 		)
 		(instances
-			(project "power_Rail"
-				(path "/aa7870c6-fc66-461c-9d29-908d06b1b5db/64ef68fa-3e19-40cc-9fb9-67d60389f594"
-					(reference "C39")
+			(project "Power_Mux"
+				(path "/c8207045-8aef-4538-bcc4-1e380c549c2c"
+					(reference "C4")
 					(unit 1)
 				)
 			)
 			(project "SuspensionBoard"
-				(path "/f9dc491a-b8c6-4623-9728-13837ac4bba3/bb9a0353-c4c7-4944-b892-c85c279a5c68/64ef68fa-3e19-40cc-9fb9-67d60389f594"
+				(path "/f9dc491a-b8c6-4623-9728-13837ac4bba3/bb9a0353-c4c7-4944-b892-c85c279a5c68/b6d6e3a7-7fd0-4579-a9e2-ac309c7dea94"
 					(reference "C39")
 					(unit 1)
@@
 		)
 		(instances
-			(project "power_Rail"
-				(path "/aa7870c6-fc66-461c-9d29-908d06b1b5db/64ef68fa-3e19-40cc-9fb9-67d60389f594"
-					(reference "R21")
+			(project "Power_Mux"
+				(path "/c8207045-8aef-4538-bcc4-1e380c549c2c"
+					(reference "R1")
 					(unit 1)
 				)
 			)
 			(project "SuspensionBoard"
-				(path "/f9dc491a-b8c6-4623-9728-13837ac4bba3/bb9a0353-c4c7-4944-b892-c85c279a5c68/64ef68fa-3e19-40cc-9fb9-67d60389f594"
+				(path "/f9dc491a-b8c6-4623-9728-13837ac4bba3/bb9a0353-c4c7-4944-b892-c85c279a5c68/b6d6e3a7-7fd0-4579-a9e2-ac309c7dea94"
 					(reference "R21")
 					(unit 1)
@@
 			)
 		)
-		(property "Value" "0.1uF"
+		(property "Value" "0.1u"
 			(at 24.5872 46.863 0)
 			(show_name no)
@@
 			)
 		)
-		(property "Mfg" "MLASH168SB7104KTNA01"
-			(at 21.59 45.72 0)
-			(hide yes)
-			(show_name no)
-			(do_not_autoplace no)
-			(effects
-				(font
-					(size 1.27 1.27)
-				)
-			)
-		)
 		(pin "1"
 		)
@@
 		)
 		(instances
-			(project "power_Rail"
-				(path "/aa7870c6-fc66-461c-9d29-908d06b1b5db/64ef68fa-3e19-40cc-9fb9-67d60389f594"
-					(reference "C36")
+			(project "Power_Mux"
+				(path "/c8207045-8aef-4538-bcc4-1e380c549c2c"
+					(reference "C1")
 					(unit 1)
 				)
 			)
 			(project "SuspensionBoard"
-				(path "/f9dc491a-b8c6-4623-9728-13837ac4bba3/bb9a0353-c4c7-4944-b892-c85c279a5c68/64ef68fa-3e19-40cc-9fb9-67d60389f594"
+				(path "/f9dc491a-b8c6-4623-9728-13837ac4bba3/bb9a0353-c4c7-4944-b892-c85c279a5c68/b6d6e3a7-7fd0-4579-a9e2-ac309c7dea94"
 					(reference "C36")
 					(unit 1)
@@
 		(dnp no)
 		(fields_autoplaced yes)
-		(property "Reference" "U5"
+		(property "Reference" "U4"
 			(at 60.96 44.45 0)
 			(show_name no)
@@
 			)
 		)
-		(property "PARTREV" "A"
-			(at 60.96 62.23 0)
-			(hide yes)
-			(show_name no)
-			(do_not_autoplace no)
-			(effects
-				(font
-					(size 1.27 1.27)
-				)
-				(justify bottom)
-			)
-		)
-		(property "STANDARD" "IPC-7351B"
-			(at 60.96 62.23 0)
-			(hide yes)
-			(show_name no)
-			(do_not_autoplace no)
-			(effects
-				(font
-					(size 1.27 1.27)
-				)
-				(justify bottom)
-			)
-		)
-		(property "MAXIMUM_PACKAGE_HEIGHT" "0.6mm"
-			(at 60.96 62.23 0)
-			(hide yes)
-			(show_name no)
-			(do_not_autoplace no)
-			(effects
-				(font
-					(size 1.27 1.27)
-				)
-				(justify bottom)
-			)
-		)
-		(property "MANUFACTURER" "Texas Instruments"
-			(at 60.96 62.23 0)
-			(hide yes)
-			(show_name no)
-			(do_not_autoplace no)
-			(effects
-				(font
-					(size 1.27 1.27)
-				)
-				(justify bottom)
-			)
-		)
 		(property "P/N" "TPS2117DRLR"
 			(at 60.96 49.53 0)
@@
 		)
 		(instances
-			(project "power_Rail"
-				(path "/aa7870c6-fc66-461c-9d29-908d06b1b5db/64ef68fa-3e19-40cc-9fb9-67d60389f594"
-					(reference "U5")
+			(project "Power_Mux"
+				(path "/c8207045-8aef-4538-bcc4-1e380c549c2c"
+					(reference "U1")
 					(unit 1)
 				)
 			)
 			(project "SuspensionBoard"
-				(path "/f9dc491a-b8c6-4623-9728-13837ac4bba3/bb9a0353-c4c7-4944-b892-c85c279a5c68/64ef68fa-3e19-40cc-9fb9-67d60389f594"
-					(reference "U5")
+				(path "/f9dc491a-b8c6-4623-9728-13837ac4bba3/bb9a0353-c4c7-4944-b892-c85c279a5c68/b6d6e3a7-7fd0-4579-a9e2-ac309c7dea94"
+					(reference "U4")
 					(unit 1)
 				)
@@
 			)
 		)
-		(property "Value" "0.1uF"
+		(property "Value" "0.1u"
 			(at 42.3672 69.723 0)
 			(show_name no)
@@
 			)
 		)
-		(property "Mfg" "MLASH168SB7104KTNA01"
-			(at 39.37 68.58 0)
-			(hide yes)
-			(show_name no)
-			(do_not_autoplace no)
-			(effects
-				(font
-					(size 1.27 1.27)
-				)
-			)
-		)
 		(pin "1"
 		)
@@
 		)
 		(instances
-			(project "power_Rail"
-				(path "/aa7870c6-fc66-461c-9d29-908d06b1b5db/64ef68fa-3e19-40cc-9fb9-67d60389f594"
-					(reference "C38")
+			(project "Power_Mux"
+				(path "/c8207045-8aef-4538-bcc4-1e380c549c2c"
+					(reference "C3")
 					(unit 1)
 				)
 			)
 			(project "SuspensionBoard"
-				(path "/f9dc491a-b8c6-4623-9728-13837ac4bba3/bb9a0353-c4c7-4944-b892-c85c279a5c68/64ef68fa-3e19-40cc-9fb9-67d60389f594"
+				(path "/f9dc491a-b8c6-4623-9728-13837ac4bba3/bb9a0353-c4c7-4944-b892-c85c279a5c68/b6d6e3a7-7fd0-4579-a9e2-ac309c7dea94"
 					(reference "C38")
 					(unit 1)
@@
 			)
 		)
-		(property "Value" "0.1uF"
+		(property "Value" "0.1u"
 			(at 38.5572 46.863 0)
 			(show_name no)
@@
 			)
 		)
-		(property "Mfg" "MLASH168SB7104KTNA01"
-			(at 35.56 45.72 0)
-			(hide yes)
-			(show_name no)
-			(do_not_autoplace no)
-			(effects
-				(font
-					(size 1.27 1.27)
-				)
-			)
-		)
 		(pin "1"
 		)
@@
 		)
 		(instances
-			(project "power_Rail"
-				(path "/aa7870c6-fc66-461c-9d29-908d06b1b5db/64ef68fa-3e19-40cc-9fb9-67d60389f594"
+			(project "Power_Mux"
+				(path "/c8207045-8aef-4538-bcc4-1e380c549c2c"
+					(reference "C2")
+					(unit 1)
+				)
+			)
+			(project "SuspensionBoard"
+				(path "/f9dc491a-b8c6-4623-9728-13837ac4bba3/bb9a0353-c4c7-4944-b892-c85c279a5c68/b6d6e3a7-7fd0-4579-a9e2-ac309c7dea94"
 					(reference "C37")
 					(unit 1)
-				)
-			)
-			(project "SuspensionBoard"
-				(path "/f9dc491a-b8c6-4623-9728-13837ac4bba3/bb9a0353-c4c7-4944-b892-c85c279a5c68/64ef68fa-3e19-40cc-9fb9-67d60389f594"
-					(reference "C37")
-					(unit 1)
