File: Hardware/power_Rail.kicad_sch (KiCad schematic)
At the start: 17 parts

Commit message: Final Changes without Footprints
Parts:
- R30: value 330 -> 2k
- R31: value 150 -> 250
Changed lines of the file:
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@@
 			)
 		)
-		(property "Value" "150"
+		(property "Value" "250"
 			(at 217.17 90.678 90)
 			(show_name no)
@@
 			)
 		)
-		(property "Value" "330"
-			(at 181.61 90.678 90)
-			(show_name no)
-			(do_not_autoplace no)
+		(property "Value" "2k"
+			(at 181.61 90.17 90)
+			(show_name no)
+			(do_not_autoplace no)
